Commit message: After nav2 integration

File: src/nav_robot/urdf/colors.xacro (robot description, xacro)
@@ -1,4 +1,5 @@
 <?xml version="1.0"?>
 <robot xmlns:xacro="http://www.ros.org/wiki/xacro" >
+    <!-- defining colors as a part of the material properties tag -->
     <material name="white">
         <color rgba="1 1 1 1"/>
@@ -13,3 +14,6 @@
         <color rgba="0 0 0 1"/>
     </material>
+    <material name="red">
+        <color rgba="1 0 0 1"/>
+    </material>
 </robot>

File: src/nav_robot/urdf/robot.urdf.xacro (robot description, xacro)
@@ -2,4 +2,6 @@
 <robot xmlns:xacro="http://www.ros.org/wiki/xacro"  name="robot">
     <xacro:include filename="robot_core.xacro" />
-    <xacro:include filename="gazebo_control.xacro" />
+    <xacro:include filename="gazebo_diff_control.xacro" />
+    <xacro:include filename="lidar.xacro" />
+    <xacro:include filename="imu.xacro" />
 </robot>

File: src/nav_robot/urdf/robot_core.xacro (robot description, xacro)
@@ -6,4 +6,12 @@
     <link name="base_link">
     </link>
+<!-- BASE FOOTPRINT (for slam) -->
+    <link name="base_footprint">
+    </link>
+    <joint name="base_footprint_joint" type="fixed">
+        <parent link="base_link"/>
+        <child link="base_footprint"/>
+        <origin xyz="0 0 0" rpy = "0 0 0"/>
+    </joint>
 <!-- CHASSIS JOINT AND LINK -->
     <joint name="chassis_joint" type="fixed">
